File: u2CEM/u2CEM.kicad_sch (KiCad schematic)
At the start: 15 parts, among them J1 PCIE_x4_10018784-10211TLF, J2 PSAS4M2130021TR

Commit message: new version
Parts:
- J1: value PCIE_x4_10018784-10211TLF -> PCIE_x4_PCIE-064-02-S-D-RA; footprint PCIe:PCIe_x4_0018784-1228695 -> U2:SAMTEC_PCIE-064-02-X-D-EMS2-BG
- J2: footprint PCIe:PSAS4M2130021TR -> U2:PSAS4M2130021TR
Connections:
- net PER1_N: now also J1.A22 (PERn[1]); no longer J1.A21 (PERp[1])
- net PER1_P: now also J1.A21 (PERp[1]); no longer J1.A22 (PERn[1])
- net PER2_N: now also J1.A26 (PERn[2]); no longer J1.A25 (PERp[2])
- net PER2_P: now also J1.A25 (PERp[2]); no longer J1.A26 (PERn[2])
Other:
- note removed: "Inverted for layout"
Changed lines of the file:
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@@
-    (effects (font (size 1.27 1.27)) (justify left bottom))
-  )
-  (text "Inverted for layout" (at 86.36 147.574 0)
     (effects (font (size 1.27 1.27)) (justify left bottom))
   )
@@
     (effects (font (size 1.27 1.27)) (justify left bottom))
   )
-  (text "Inverted for layout" (at 86.36 137.668 0)
-    (effects (font (size 1.27 1.27)) (justify left bottom))
-  )
   (label "SMBDAT" (at 184.912 94.742 0)
     (effects (font (size 1.27 1.27)) (justify left bottom))
@@
     (effects (font (size 1.27 1.27)) (justify left bottom))
   )
-  (label "PER1_N" (at 110.744 135.382 0)
+  (label "PER1_P" (at 110.744 135.382 0)
     (effects (font (size 1.27 1.27)) (justify left bottom))
   )
@@
     (effects (font (size 1.27 1.27)) (justify left bottom))
   )
-  (label "PER2_N" (at 111.252 145.542 0)
+  (label "PER2_P" (at 111.252 145.542 0)
     (effects (font (size 1.27 1.27)) (justify left bottom))
   )
@@
     (effects (font (size 1.27 1.27)) (justify left bottom))
   )
-  (label "PER2_P" (at 111.252 148.082 0)
+  (label "PER2_N" (at 111.252 148.082 0)
     (effects (font (size 1.27 1.27)) (justify left bottom))
   )
@@
     (effects (font (size 1.27 1.27)) (justify left bottom))
   )
-  (label "PER1_P" (at 110.49 137.922 0)
+  (label "PER1_N" (at 110.49 137.922 0)
     (effects (font (size 1.27 1.27)) (justify left bottom))
   )
@@
     (property "Reference" "J2" (id 0) (at 291.338 66.802 0))
     (property "Value" "PSAS4M2130021TR" (id 1) (at 291.338 69.342 0))
-    (property "Footprint" "PCIe:PSAS4M2130021TR" (id 2) (at 268.478 71.882 0)
+    (property "Footprint" "U2:PSAS4M2130021TR" (id 2) (at 268.478 71.882 0)
       (effects (font (size 1.27 1.27)) hide)
     )
@@
   (symbol (lib_id "PCIeLib:PCIE_x4_10018784-10211TLF") (at 131.064 78.232 0) (unit 1)
     (in_bom yes) (on_board yes) (fields_autoplaced)
-    (property "Reference" "J1" (id 0) (at 150.114 72.898 0))
-    (property "Value" "PCIE_x4_10018784-10211TLF" (id 1) (at 150.114 75.438 0))
-    (property "Footprint" "PCIe:PCIe_x4_0018784-1228695" (id 2) (at 131.064 78.232 0)
+    (property "Reference" "J1" (id 0) (at 150.114 76.2 0))
+    (property "Value" "PCIE_x4_PCIE-064-02-S-D-RA" (id 1) (at 150.114 78.74 0))
+    (property "Footprint" "U2:SAMTEC_PCIE-064-02-X-D-EMS2-BG" (id 2) (at 131.064 78.232 0)
       (effects (font (size 1.27 1.27)) hide)
     )
@@
     )
     (path "/f6047208-a400-4c9b-b580-6127a217a3b4"
-      (reference "J1") (unit 1) (value "PCIE_x4_10018784-10211TLF") (footprint "PCIe:PCIe_x4_0018784-1228695")
+      (reference "J1") (unit 1) (value "PCIE_x4_PCIE-064-02-S-D-RA") (footprint "U2:SAMTEC_PCIE-064-02-X-D-EMS2-BG")
     )
     (path "/1c34329e-a374-4c99-aa52-979381eab278"
-      (reference "J2") (unit 1) (value "PSAS4M2130021TR") (footprint "PCIe:PSAS4M2130021TR")
+      (reference "J2") (unit 1) (value "PSAS4M2130021TR") (footprint "U2:PSAS4M2130021TR")
     )
     (path "/827d739e-6bd1-4c48-99f2-05ca99dcfa37"
