File: u2CEM.kicad_sch (KiCad schematic)
At the start: 15 parts, among them J1 PCIE_x4_PCIE-064-02-S-D-RA, J2 PSAS4M2130021TR

Commit message: updating mech model for clearance on Cosmo U.2 guide tabs
Parts:
- J1: value PCIE_x4_PCIE-064-02-S-D-RA -> PCIE-064-02-F-D-EMS2-BG

Commit message: initial quote request to Sierra
Parts:
- D1, D2: MFG (none) -> Lite-On Inc.; MPN (none) -> LTST-C193KSKT-5A
- J1: MFG (none) -> Samtec; MPN (none) -> PCIE-064-02-F-D-EMS2-BG
- J2: MFG (none) -> Amphenol; MPN (none) -> PSAS4M2130021TR
- R1, R10, R11, R2, R3, R4, R6, R7: now not fitted
- R5: MFG (none) -> Yageo; MPN (none) -> RC0603JR-070RL
- R8: value 5k -> 5.11k; MFG (none) -> Yageo; MPN (none) -> RC0603FR-075K11L
- R9: MFG (none) -> Yageo; MPN (none) -> RC0603FR-071K4L
Other:
- title: (none) -> 913-0000114 K.2
Changed lines of the file:
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@@
 	(generator_version "9.0")
 	(paper "USLedger")
+	(title_block
+		(title "913-0000114 K.2")
+		(date "2026-03-10")
+		(rev "Rev 1")
+	)
 	(text "CEM x4 Socket"
 		(exclude_from_sim no)
@@
 		(in_bom yes)
 		(on_board yes)
-		(dnp no)
+		(dnp yes)
 		(property "Reference" "R3"
 			(at 204.978 95.504 0)
@@
 			)
 		)
+		(property "MPN" "PSAS4M2130021TR"
+			(at 268.478 71.882 0)
+			(effects
+				(font
+					(size 1.27 1.27)
+				)
+				(hide yes)
+			)
+		)
+		(property "MFG" "Amphenol"
+			(at 268.478 71.882 0)
+			(effects
+				(font
+					(size 1.27 1.27)
+				)
+				(hide yes)
+			)
+		)
 		(pin "E1"
 		)
@@
 			)
 		)
+		(property "MPN" "LTST-C193KSKT-5A"
+			(at 45.466 146.812 90)
+			(effects
+				(font
+					(size 1.27 1.27)
+				)
+				(hide yes)
+			)
+		)
+		(property "MFG" "Lite-On Inc."
+			(at 45.466 146.812 90)
+			(effects
+				(font
+					(size 1.27 1.27)
+				)
+				(hide yes)
+			)
+		)
 		(pin "1"
 		)
@@
 		(in_bom yes)
 		(on_board yes)
-		(dnp no)
+		(dnp yes)
 		(property "Reference" "R7"
 			(at 238.506 134.366 0)
@@
 		(in_bom yes)
 		(on_board yes)
-		(dnp no)
+		(dnp yes)
 		(property "Reference" "R11"
 			(at 232.664 164.592 0)
@@
 		(in_bom yes)
 		(on_board yes)
-		(dnp no)
+		(dnp yes)
 		(fields_autoplaced yes)
 		(property "Reference" "R2"
@@
 			)
 		)
+		(property "MPN" "RC0603FR-071K4L"
+			(at 55.372 137.668 0)
+			(effects
+				(font
+					(size 1.27 1.27)
+				)
+				(hide yes)
+			)
+		)
+		(property "MFG" "Yageo"
+			(at 55.372 137.668 0)
+			(effects
+				(font
+					(size 1.27 1.27)
+				)
+				(hide yes)
+			)
+		)
 		(pin "1"
 		)
@@
 		(in_bom yes)
 		(on_board yes)
-		(dnp no)
+		(dnp yes)
 		(property "Reference" "R4"
 			(at 210.566 95.504 0)
@@
 		(in_bom yes)
 		(on_board yes)
-		(dnp no)
+		(dnp yes)
 		(property "Reference" "R6"
 			(at 238.506 124.206 0)
@@
 		(in_bom yes)
 		(on_board yes)
-		(dnp no)
+		(dnp yes)
 		(property "Reference" "R1"
 			(at 199.39 95.504 0)
@@
 			)
 		)
+		(property "MPN" "LTST-C193KSKT-5A"
+			(at 55.372 147.066 90)
+			(effects
+				(font
+					(size 1.27 1.27)
+				)
+				(hide yes)
+			)
+		)
+		(property "MFG" "Lite-On Inc."
+			(at 55.372 147.066 90)
+			(effects
+				(font
+					(size 1.27 1.27)
+				)
+				(hide yes)
+			)
+		)
 		(pin "1"
 		)
@@
 			)
 		)
+		(property "MPN" "RC0603JR-070RL"
+			(at 230.124 130.302 90)
+			(effects
+				(font
+					(size 1.27 1.27)
+				)
+				(hide yes)
+			)
+		)
+		(property "MFG" "Yageo"
+			(at 230.124 130.302 90)
+			(effects
+				(font
+					(size 1.27 1.27)
+				)
+				(hide yes)
+			)
+		)
 		(pin "1"
 		)
@@
 		(fields_autoplaced yes)
 		(property "Reference" "R8"
-			(at 48.006 136.6519 0)
+			(at 48.26 136.6519 0)
 			(effects
 				(font
@@
 			)
 		)
-		(property "Value" "5k"
-			(at 48.006 139.1919 0)
+		(property "Value" "5.11k"
+			(at 48.26 139.1919 0)
 			(effects
 				(font
@@
 			)
 		)
+		(property "MPN" "RC0603FR-075K11L"
+			(at 45.466 137.922 0)
+			(effects
+				(font
+					(size 1.27 1.27)
+				)
+				(hide yes)
+			)
+		)
+		(property "MFG" "Yageo"
+			(at 45.466 137.922 0)
+			(effects
+				(font
+					(size 1.27 1.27)
+				)
+				(hide yes)
+			)
+		)
 		(pin "1"
 		)
@@
 			)
 		)
+		(property "MPN" "PCIE-064-02-F-D-EMS2-BG"
+			(at 131.064 78.232 0)
+			(effects
+				(font
+					(size 1.27 1.27)
+				)
+				(hide yes)
+			)
+		)
+		(property "MFG" "Samtec"
+			(at 131.064 78.232 0)
+			(effects
+				(font
+					(size 1.27 1.27)
+				)
+				(hide yes)
+			)
+		)
 		(pin "A01"
 		)
@@
 		(in_bom yes)
 		(on_board yes)
-		(dnp no)
+		(dnp yes)
 		(property "Reference" "R10"
 			(at 232.664 154.432 0)
